Commit message: 功能：增加 Gazebo 原生六轴运行环境

File: src/dummy-ros2_description/urdf/dummy-ros2.xacro (robot description, xacro)
@@ -17,7 +17,7 @@
   </visual>
   <collision>
-    <origin xyz="0 0 0" rpy="0 0 0"/>
-    <geometry>
-      <mesh filename="file://$(find dummy-ros2_description)/meshes/base_link.stl" scale="0.001 0.001 0.001"/>
+    <origin xyz="-0.019225 -0.005523 0.054184" rpy="0 0 0"/>
+    <geometry>
+      <box size="0.1 0.11 0.099"/>
     </geometry>
   </collision>
@@ -37,7 +37,7 @@
   </visual>
   <collision>
-    <origin xyz="0.019225 0.000523 -0.100684" rpy="0 0 0"/>
-    <geometry>
-      <mesh filename="file://$(find dummy-ros2_description)/meshes/link1_1_1.stl" scale="0.001 0.001 0.001"/>
+    <origin xyz="0.00095 0.009 0.017749" rpy="0 0 0"/>
+    <geometry>
+      <box size="0.0629 0.079 0.048499"/>
     </geometry>
   </collision>
@@ -57,7 +57,7 @@
   </visual>
   <collision>
-    <origin xyz="0.034725 -0.034477 -0.129184" rpy="0 0 0"/>
-    <geometry>
-      <mesh filename="file://$(find dummy-ros2_description)/meshes/link2_1_1.stl" scale="0.001 0.001 0.001"/>
+    <origin xyz="0.021575 0.001501 0.073002" rpy="0 0 0"/>
+    <geometry>
+      <box size="0.05585 0.050998 0.193995"/>
     </geometry>
   </collision>
@@ -77,7 +77,7 @@
   </visual>
   <collision>
-    <origin xyz="-0.001925 -0.034477 -0.275184" rpy="0 0 0"/>
-    <geometry>
-      <mesh filename="file://$(find dummy-ros2_description)/meshes/link3_1_1.stl" scale="0.001 0.001 0.001"/>
+    <origin xyz="-0.011975 -0.014252 0.04735" rpy="0 0 0"/>
+    <geometry>
+      <box size="0.05115 0.051495 0.1177"/>
     </geometry>
   </collision>
@@ -97,7 +97,7 @@
   </visual>
   <collision>
-    <origin xyz="0.016625 -0.024477 -0.327184" rpy="0 0 0"/>
-    <geometry>
-      <mesh filename="file://$(find dummy-ros2_description)/meshes/link4_1_1.stl" scale="0.001 0.001 0.001"/>
+    <origin xyz="-0.0027 0.0755 0" rpy="0 0 0"/>
+    <geometry>
+      <box size="0.039 0.151 0.048"/>
     </geometry>
   </collision>
@@ -117,7 +117,7 @@
   </visual>
   <collision>
-    <origin xyz="-0.000175 -0.151477 -0.327184" rpy="0 0 0"/>
-    <geometry>
-      <mesh filename="file://$(find dummy-ros2_description)/meshes/link5_1_1.stl" scale="0.001 0.001 0.001"/>
+    <origin xyz="-0.0148 0.030004 0" rpy="0 0 0"/>
+    <geometry>
+      <box size="0.048 0.093992 0.036"/>
     </geometry>
   </collision>
@@ -137,7 +137,7 @@
   </visual>
   <collision>
-    <origin xyz="0.018331 -0.228477 -0.327078" rpy="0 0 0"/>
-    <geometry>
-      <mesh filename="file://$(find dummy-ros2_description)/meshes/link6_1_1.stl" scale="0.001 0.001 0.001"/>
+    <origin xyz="-0.000001 0.0015 -0.000002" rpy="0 0 0"/>
+    <geometry>
+      <box size="0.022997 0.003 0.022996"/>
     </geometry>
   </collision>

Commit message: 维护：保存已验证机械臂功能源码基线

File: src/dummy-ros2_description/urdf/dummy-ros2.xacro (robot description, xacro)
@@ -9,6 +9,6 @@
   <xacro:arg name="Joint4_lower" default="-3.141592653589793"/>
   <xacro:arg name="Joint4_upper" default="3.141592653589793"/>
-  <xacro:arg name="Joint5_lower" default="-2.0943951023931953"/>
-  <xacro:arg name="Joint5_upper" default="2.0943951023931953"/>
+  <xacro:arg name="Joint5_lower" default="-1.7453292519943295"/>
+  <xacro:arg name="Joint5_upper" default="1.7453292519943295"/>
   <xacro:arg name="Joint6_lower" default="-12.566370614359172"/>
   <xacro:arg name="Joint6_upper" default="12.566370614359172"/>
@@ -29,7 +29,7 @@
   </visual>
   <collision>
-    <origin xyz="-0.019225 -0.005523 0.054184" rpy="0 0 0"/>
-    <geometry>
-      <box size="0.1 0.11 0.099"/>
+    <origin xyz="0 0 0" rpy="0 0 0"/>
+    <geometry>
+      <mesh filename="file://$(find dummy-ros2_description)/meshes/base_link.stl" scale="0.001 0.001 0.001"/>
     </geometry>
   </collision>
@@ -49,7 +49,7 @@
   </visual>
   <collision>
-    <origin xyz="0.00095 0.009 0.017749" rpy="0 0 0"/>
-    <geometry>
-      <box size="0.0629 0.079 0.048499"/>
+    <origin xyz="0.019225 0.000523 -0.100684" rpy="0 0 0"/>
+    <geometry>
+      <mesh filename="file://$(find dummy-ros2_description)/meshes/link1_1_1.stl" scale="0.001 0.001 0.001"/>
     </geometry>
   </collision>
@@ -69,7 +69,7 @@
   </visual>
   <collision>
-    <origin xyz="0.021575 0.001501 0.073002" rpy="0 0 0"/>
-    <geometry>
-      <box size="0.05585 0.050998 0.193995"/>
+    <origin xyz="0.034725 -0.034477 -0.129184" rpy="0 0 0"/>
+    <geometry>
+      <mesh filename="file://$(find dummy-ros2_description)/meshes/link2_1_1.stl" scale="0.001 0.001 0.001"/>
     </geometry>
   </collision>
@@ -89,7 +89,7 @@
   </visual>
   <collision>
-    <origin xyz="-0.011975 -0.014252 0.04735" rpy="0 0 0"/>
-    <geometry>
-      <box size="0.05115 0.051495 0.1177"/>
+    <origin xyz="-0.001925 -0.034477 -0.275184" rpy="0 0 0"/>
+    <geometry>
+      <mesh filename="file://$(find dummy-ros2_description)/meshes/link3_1_1.stl" scale="0.001 0.001 0.001"/>
     </geometry>
   </collision>
@@ -109,7 +109,7 @@
   </visual>
   <collision>
-    <origin xyz="-0.0027 0.0755 0" rpy="0 0 0"/>
-    <geometry>
-      <box size="0.039 0.151 0.048"/>
+    <origin xyz="0.016625 -0.024477 -0.327184" rpy="0 0 0"/>
+    <geometry>
+      <mesh filename="file://$(find dummy-ros2_description)/meshes/link4_1_1.stl" scale="0.001 0.001 0.001"/>
     </geometry>
   </collision>
@@ -129,7 +129,7 @@
   </visual>
   <collision>
-    <origin xyz="-0.0148 0.030004 0" rpy="0 0 0"/>
-    <geometry>
-      <box size="0.048 0.093992 0.036"/>
+    <origin xyz="-0.000175 -0.151477 -0.327184" rpy="0 0 0"/>
+    <geometry>
+      <mesh filename="file://$(find dummy-ros2_description)/meshes/link5_1_1.stl" scale="0.001 0.001 0.001"/>
     </geometry>
   </collision>
@@ -149,7 +149,7 @@
   </visual>
   <collision>
-    <origin xyz="-0.000001 0.0015 -0.000002" rpy="0 0 0"/>
-    <geometry>
-      <box size="0.022997 0.003 0.022996"/>
+    <origin xyz="0.018331 -0.228477 -0.327078" rpy="0 0 0"/>
+    <geometry>
+      <mesh filename="file://$(find dummy-ros2_description)/meshes/link6_1_1.stl" scale="0.001 0.001 0.001"/>
     </geometry>
   </collision>
@@ -177,6 +177,7 @@
     velocity="3.15" />
 </joint>
+<!-- Display: CAD q3=0 is the 7 pose; canonical Home q3=90 uses +X90 with axis -X. All ROS viewers must load this same file. -->
 <joint name="Joint3" type="revolute">
-  <origin xyz="0.03665 0.0 0.146" rpy="0 0 0"/>
+  <origin xyz="0.03665 0.0 0.146" rpy="1.5707963267948966 0 0"/>
   <parent link="link2_1_1"/>
   <child link="link3_1_1"/>

File: src/dummy-ros2_description/urdf/dummy_reference_chain.urdf (robot description, URDF)
Before this commit: robot dummy_reference_chain, 13 links, 12 joints
Joints:
- joint Joint5: limit lower=-2.0943951023931953 upper=2.0943951023931953 effort=1 velocity=0.25 -> lower=-1.7453292519943295 upper=1.7453292519943295 effort=1 velocity=0.25

File: src/dummy-ros2_description/urdf/dummy_reference_chain.xacro (robot description, xacro)
@@ -52,5 +52,5 @@
     <joint name="${prefix}Joint5" type="revolute">
       <parent link="${prefix}reference_link4"/><child link="${prefix}reference_joint5"/>
-      <axis xyz="0 0 1"/><limit lower="-2.0943951023931953" upper="2.0943951023931953" effort="1" velocity="0.25"/>
+      <axis xyz="0 0 1"/><limit lower="-1.7453292519943295" upper="1.7453292519943295" effort="1" velocity="0.25"/>
     </joint>
     <joint name="${prefix}Joint5_dh" type="fixed">

File: src/dummy_bringup/config/dummy_ref_real_6dof.urdf.xacro (robot description, xacro)
@@ -20,4 +20,5 @@
   <xacro:arg name="max_state_age_us" default=""/>
   <xacro:arg name="heartbeat_stop_budget_us" default=""/>
+  <xacro:arg name="stop_confirmation_timeout_us" default="0"/>
   <xacro:arg name="raw_evidence_path" default=""/>
   <xacro:macro name="required_param" params="key value">
@@ -45,4 +46,5 @@
       <xacro:required_param key="max_state_age_us" value="$(arg max_state_age_us)"/>
       <xacro:required_param key="heartbeat_stop_budget_us" value="$(arg heartbeat_stop_budget_us)"/>
+      <param name="stop_confirmation_timeout_us">$(arg stop_confirmation_timeout_us)</param>
       <xacro:if value="${bool(xacro.arg('raw_evidence_path'))}">
         <param name="raw_evidence_path">$(arg raw_evidence_path)</param>
